Commit message: Fully working diff drive controller with urdf

File: src/diffdrive_jetbot/description/ros2_control/diffbot.ros2_control.xacro (robot description, xacro)
@@ -5,6 +5,6 @@
       <hardware>
         <plugin>diffdrive_jetbot/DiffDriveJetbotHardware</plugin>
-        <param name="left_wheel_name">left_wheel_joint</param>
-        <param name="right_wheel_name">right_wheel_joint</param>
+        <param name="left_wheel_name">left_wheel_continuous_joint</param>
+        <param name="right_wheel_name">right_wheel_continuous_joint</param>
         <param name="device">/dev/ttyUSB0</param>
         <param name="baud_rate">115200</param>
@@ -20,10 +20,10 @@
         <param name="pid_d">0.5</param>
       </hardware>
-      <joint name="${prefix}left_wheel_joint">
+      <joint name="${prefix}left_wheel_continuous_joint">
         <command_interface name="velocity"/>
         <state_interface name="position"/>
         <state_interface name="velocity"/>
       </joint>
-      <joint name="${prefix}right_wheel_joint">
+      <joint name="${prefix}right_wheel_continuous_joint">
         <command_interface name="velocity"/>
         <state_interface name="position"/>

File: src/diffdrive_jetbot/description/urdf/diffbot_description.urdf.xacro (robot description, xacro)
@@ -2,160 +2,329 @@
 <robot xmlns:xacro="http://www.ros.org/wiki/xacro">
   <xacro:macro name="diffbot" params="prefix">
-  <!-- Constants for robot dimensions -->
-  <xacro:property name="PI" value="3.1415926535897931"/>
-  <xacro:property name="base_mass" value="0.3" /> <!-- arbitrary value for base mass -->
-  <xacro:property name="base_width" value="0.1" />
-  <xacro:property name="base_length" value="0.1" />
-  <xacro:property name="base_height" value="0.05" />
-  <xacro:property name="wheel_mass" value="0.3" /> <!-- arbitrary value for wheel mass -->
-  <xacro:property name="wheel_len" value="0.020" />
-  <xacro:property name="wheel_radius" value="0.015" />
-  <xacro:property name="caster_wheel_mass" value="0.1" /> <!-- arbitrary value for caster wheel mass -->
-  <xacro:property name="caster_wheel_radius" value="0.015" />
-  <xacro:property name="z_offset" value="-${base_height/2}" /> <!-- Space btw top of beam and the each joint -->
-  <!-- Base Link -->
-  <link name="${prefix}base_link">
-    <collision>
-      <origin xyz="0 0 0" rpy="0 0 0"/>
-      <geometry>
-        <box size="${base_width} ${base_length} ${base_height}"/>
-      </geometry>
-    </collision>
-    <visual>
-      <origin xyz="0 0 ${base_height/2}" rpy="0 0 0"/>
-      <geometry>
-        <box size="${base_width} ${base_length} ${base_height}"/>
-      </geometry>
-      <material name="orange"/>
-    </visual>
-    <inertial>
-      <origin xyz="0 0 0" rpy="0 0 0"/>
-      <mass value="${base_mass}"/>
-      <inertia
-        ixx="${base_mass / 12.0 * (base_length*base_length + base_height*base_height)}" ixy="0.0" ixz="0.0"
-        iyy="${base_mass / 12.0 * (base_height*base_height + base_width*base_width)}" iyz="0.0"
-        izz="${base_mass / 12.0 * (base_width*base_width + base_length*base_length)}"/>
-      </inertial>
-    </link>
-    <joint name="${prefix}left_wheel_joint" type="continuous">
-      <parent link="${prefix}base_link"/>
-      <child link="${prefix}left_wheel"/>
-      <origin xyz="0 -${base_width/2} ${z_offset}" rpy="0 0 0"/>
-      <axis xyz="0 1 0"/>
-      <dynamics damping="0.2"/>
-    </joint>
-    <!-- left wheel Link -->
-    <link name="${prefix}left_wheel">
-      <collision>
-        <origin xyz="0 0 0" rpy="${PI/2} 0 0"/>
-        <geometry>
-          <cylinder length="${wheel_len}" radius="${wheel_radius}"/>
-        </geometry>
-      </collision>
-      <visual>
-        <origin xyz="0 0 0" rpy="${PI/2} 0 0"/>
-        <geometry>
-          <cylinder length="${wheel_len}" radius="${wheel_radius}"/>
-        </geometry>
-        <material name="black"/>
-      </visual>
-      <inertial>
-        <origin xyz="0 0 0" rpy="${PI/2} 0 0"/>
-        <mass value="${wheel_mass}"/>
-        <inertia
-          ixx="${wheel_mass / 12.0 * (3*wheel_radius + wheel_len*wheel_len)}" ixy="0.0" ixz="0.0"
-          iyy="${wheel_mass / 12.0 * wheel_radius*wheel_radius}" iyz="0.0"
-          izz="${wheel_mass / 12.0 * wheel_radius*wheel_radius}"/>
-        </inertial>
-      </link>
-    <joint name="${prefix}right_wheel_joint" type="continuous">
-      <parent link="${prefix}base_link"/>
-      <child link="${prefix}right_wheel"/>
-      <origin xyz="0 ${base_width/2} ${z_offset}" rpy="0 0 0"/>
-      <axis xyz="0 1 0"/>
-      <dynamics damping="0.2"/>
-    </joint>
-    <!-- right wheel Link -->
-    <link name="${prefix}right_wheel">
-      <collision>
-        <origin xyz="0 0 0" rpy="${PI/2} 0 0"/>
-        <geometry>
-          <cylinder length="${wheel_len}" radius="${wheel_radius}"/>
-        </geometry>
-      </collision>
-      <visual>
-        <origin xyz="0 0 0" rpy="${PI/2} 0 0"/>
-        <geometry>
-          <cylinder length="${wheel_len}" radius="${wheel_radius}"/>
-        </geometry>
-        <material name="black"/>
-      </visual>
-      <inertial>
-        <origin xyz="0 0 0" rpy="${PI/2} 0 0"/>
-        <mass value="${wheel_mass}"/>
-        <inertia
-          ixx="${wheel_mass / 12.0 * (3*wheel_radius + wheel_len*wheel_len)}" ixy="0.0" ixz="0.0"
-          iyy="${wheel_mass / 12.0 * wheel_radius*wheel_radius}" iyz="0.0"
-          izz="${wheel_mass / 12.0 * wheel_radius*wheel_radius}"/>
-        </inertial>
-      </link>
-    <joint name="${prefix}caster_frontal_wheel_joint" type="fixed">
-      <parent link="${prefix}base_link"/>
-      <child link="${prefix}caster_frontal_wheel"/>
-      <origin xyz="${base_width/2 - caster_wheel_radius} 0 ${z_offset}" rpy="0 0 0"/>
-    </joint>
-    <!-- caster frontal wheel Link -->
-    <link name="${prefix}caster_frontal_wheel">
-      <collision>
-        <origin xyz="0 0 0" rpy="0 0 0"/>
-        <geometry>
-          <sphere radius="${caster_wheel_radius}"/>
-        </geometry>
-      </collision>
-      <visual>
-        <origin xyz="0 0 0" rpy="0 0 0"/>
-        <geometry>
-          <sphere radius="${caster_wheel_radius}"/>
-        </geometry>
-        <material name="white"/>
-      </visual>
-      <inertial>
-        <origin xyz="0 0 0" rpy="0 0 0"/>
-        <mass value="${caster_wheel_mass}"/>
-        <inertia
-          ixx="${caster_wheel_mass * 0.4 * (caster_wheel_radius * caster_wheel_radius)}" ixy="0.0" ixz="0.0"
-          iyy="${caster_wheel_mass * 0.4 * (caster_wheel_radius * caster_wheel_radius)}" iyz="0.0"
-          izz="${caster_wheel_mass * 0.4 * (caster_wheel_radius * caster_wheel_radius)}"/>
-        </inertial>
-      </link>
-    <joint name="${prefix}caster_rear_wheel_joint" type="fixed">
-      <parent link="${prefix}base_link"/>
-      <child link="${prefix}caster_rear_wheel"/>
-      <origin xyz="${-base_width/2 + caster_wheel_radius} 0 ${z_offset}" rpy="0 0 0"/>
-    </joint>
-    <!-- caster rear wheel Link -->
-    <link name="${prefix}caster_rear_wheel">
-      <collision>
-        <origin xyz="0 0 0" rpy="0 0 0"/>
-        <geometry>
-          <sphere radius="${caster_wheel_radius}"/>
-        </geometry>
-      </collision>
-      <visual>
-        <origin xyz="0 0 0" rpy="0 0 0"/>
-        <geometry>
-          <sphere radius="${caster_wheel_radius}"/>
-        </geometry>
-        <material name="white"/>
-      </visual>
-      <inertial>
-        <origin xyz="0 0 0" rpy="0 0 0"/>
-        <mass value="${caster_wheel_mass}"/>
-        <inertia
-          ixx="${caster_wheel_mass * 0.4 * (caster_wheel_radius * caster_wheel_radius)}" ixy="0.0" ixz="0.0"
-          iyy="${caster_wheel_mass * 0.4 * (caster_wheel_radius * caster_wheel_radius)}" iyz="0.0"
-          izz="${caster_wheel_mass * 0.4 * (caster_wheel_radius * caster_wheel_radius)}"/>
-        </inertial>
-      </link>
+  <link name="${prefix}base_link"/>
+  <!-- Was base_link, now body_link -->
+  <link
+    name="${prefix}body_link">
+    <inertial>
+      <origin
+        xyz="-0.025609 0.0093176 0.034957"
+        rpy="0 0 0" />
+      <mass
+        value="2" />
+      <inertia
+        ixx="0.0016616"
+        ixy="-5.2805E-05"
+        ixz="-3.0797E-06"
+        iyy="0.0024755"
+        iyz="-1.1469E-06"
+        izz="0.0030448" />
+    </inertial>
+    <visual>
+      <origin
+        xyz="0 0 0"
+        rpy="0 0 0" />
+      <geometry>
+        <mesh
+          filename="package://diffdrive_jetbot/description/meshes/body_link.STL" />
+      </geometry>
+      <material
+        name="">
+        <color
+          rgba="0.61176 0.65882 0.67059 1" />
+      </material>
+    </visual>
+    <collision>
+      <origin
+        xyz="0 0 0"
+        rpy="0 0 0" />
+      <geometry>
+        <mesh
+          filename="package://diffdrive_jetbot/description/meshes/body_link.STL" />
+      </geometry>
+    </collision>
+  </link>
+  <!-- Fixed joint between base_link and body_link -->
+  <joint
+    name="${prefix}body_fix_joint"
+    type="fixed">
+    <origin
+      xyz="0 0 0.035"
+      rpy="-1.5708 0 0" />
+    <parent
+      link="${prefix}base_link" />
+    <child
+      link="${prefix}body_link" />
+    <axis
+      xyz="0 0 0" />
+  </joint>
+  <link
+    name="${prefix}caster_ball_link">
+    <inertial>
+      <origin
+        xyz="-1.8666E-06 -8.4152E-07 -0.0059479"
+        rpy="0 0 0" />
+      <mass
+        value="0.011917" />
+      <inertia
+        ixx="2.5586E-07"
+        ixy="6.7546E-11"
+        ixz="3.0679E-11"
+        iyy="1.8138E-07"
+        iyz="1.7478E-14"
+        izz="2.6388E-07" />
+    </inertial>
+    <visual>
+      <origin
+        xyz="0 0 0"
+        rpy="0 0 0" />
+      <geometry>
+        <mesh
+          filename="package://diffdrive_jetbot/description/meshes/caster_ball_link.STL" />
+      </geometry>
+      <material
+        name="">
+        <color
+          rgba="0.61176 0.65882 0.67059 1" />
+      </material>
+    </visual>
+    <collision>
+      <origin
+        xyz="0 0 0"
+        rpy="0 0 0" />
+      <geometry>
+        <mesh
+          filename="package://diffdrive_jetbot/description/meshes/caster_ball_link.STL" />
+      </geometry>
+    </collision>
+  </link>
+  <joint
+    name="${prefix}caster_ball_fix_joint"
+    type="fixed">
+    <origin
+      xyz="-0.083 0.0208 0"
+      rpy="-1.5708 0 3.1416" />
+    <parent
+      link="${prefix}body_link" />
+    <child
+      link="${prefix}caster_ball_link" />
+    <axis
+      xyz="0 0 0" />
+  </joint>
+  <link
+    name="${prefix}camera_link">
+    <inertial>
+      <origin
+        xyz="7.2979E-05 -0.0036847 -0.0021354"
+        rpy="0 0 0" />
+      <mass
+        value="0.068956" />
+      <inertia
+        ixx="2.4451E-06"
+        ixy="1.5517E-12"
+        ixz="-1.8066E-08"
+        iyy="3.8509E-06"
+        iyz="1.5741E-11"
+        izz="2.7785E-06" />
+    </inertial>
+    <visual>
+      <origin
+        xyz="0 0 0"
+        rpy="0 0 0" />
+      <geometry>
+        <mesh
+          filename="package://diffdrive_jetbot/description/meshes/camera_link.STL" />
+      </geometry>
+      <material
+        name="">
+        <color
+          rgba="0.61176 0.65882 0.67059 1" />
+      </material>
+    </visual>
+    <collision>
+      <origin
+        xyz="0 0 0"
+        rpy="0 0 0" />
+      <geometry>
+        <mesh
+          filename="package://diffdrive_jetbot/description/meshes/camera_link.STL" />
+      </geometry>
+    </collision>
+  </link>
+  <joint
+    name="${prefix}camera_fix_joint"
+    type="fixed">
+    <origin
+      xyz="0.053557 -0.057568 0"
+      rpy="1.9199 -1.5708 3.1416" />
+    <parent
+      link="${prefix}body_link" />
+    <child
+      link="${prefix}camera_link" />
+    <axis
+      xyz="0 0 0" />
+  </joint>
+  <link
+    name="${prefix}lidar_link">
+    <inertial>
+      <origin
+        xyz="-0.0065398705841951 0.000690713934940602 0.0309531855778308"
+        rpy="0 0 0" />
+      <mass
+        value="0.564294014597891" />
+      <inertia
+        ixx="0.000142259766419758"
+        ixy="-2.48879198210457E-06"
+        ixz="2.55066150802879E-06"
+        iyy="0.000186813526823412"
+        iyz="8.53957008589798E-08"
+        izz="0.000308569075147343" />
+    </inertial>
+    <visual>
+      <!-- Shift mesh down by 0.045 along z to compensate for frame shift up -->
+      <origin
+        xyz="0 0 -0.045 "
+        rpy="0 0 0" />
+      <geometry>
+        <mesh
+          filename="package://diffdrive_jetbot/description/meshes/lidar_link.STL" />
+      </geometry>
+      <material
+        name="">
+        <color
+          rgba="0.611764705882353 0.658823529411765 0.670588235294118 1" />
+      </material>
+    </visual>
+    <collision>
+      <!-- Shift mesh down by 0.045 along z to compensate for frame shift up -->
+      <origin
+        xyz="0 0 -0.045"
+        rpy="0 0 0" />
+      <geometry>
+        <mesh
+          filename="package://diffdrive_jetbot/description/meshes/lidar_link.STL" />
+      </geometry>
+    </collision>
+  </link>
+  <joint
+    name="${prefix}lidar_fix_joint"
+    type="fixed">
+    <!-- Raise lidar_link frame by 0.045 along z -->
+     <!-- xyz="-0.011026 -0.10618-0.045 0 " -->
+    <origin
+      xyz="-0.011026 -0.1512 0 "
+      rpy="1.5708 0 0" />
+    <parent
+      link="${prefix}body_link" />
+    <child
+      link="${prefix}lidar_link" />
+    <axis
+      xyz="0 0 0" />
+  </joint>
+  <link
+    name="${prefix}left_wheel_link">
+    <inertial>
+      <origin
+        xyz="-3.04495944265183E-05 0.0183179040454366 -1.07396547774597E-07"
+        rpy="0 0 0" />
+      <mass
+        value="0.388137366198046" />
+      <inertia
+        ixx="0.000163568162825962"
+        ixy="-1.71522947947033E-07"
+        ixz="-2.55253489205791E-08"
+        iyy="0.000281670214792073"
+        iyz="-1.06397401901507E-09"
+        izz="0.000163656330155147" />
+    </inertial>
+    <visual>
+      <origin
+        xyz="0 0 0"
+        rpy="0 0 0" />
+      <geometry>
+        <mesh
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
Commit message: Fully working slam example

File: src/diffdrive_jetbot/description/ros2_control/diffbot.ros2_control.xacro (robot description, xacro)
@@ -9,5 +9,5 @@
         <param name="device">/dev/ttyMOTOR</param>
         <param name="baud_rate">115200</param>
-        <param name="timeout_ms">200</param>
+        <param name="timeout_ms">20</param>
         <param name="mtype">1</param>
         <param name="deadzone">1600</param>

File: src/diffdrive_jetbot/description/urdf/diffbot.urdf.xacro (robot description, xacro)
@@ -10,4 +10,4 @@
   <xacro:diffbot prefix="$(arg prefix)" />
   <xacro:diffbot_ros2_control
-    name="DiffBot" prefix="$(arg prefix)" />
+    name="DiffBot" prefix="$(arg prefix)"/>
 </robot>

File: src/diffdrive_jetbot/description/urdf/diffbot_description.urdf.xacro (robot description, xacro)
@@ -2,8 +2,7 @@
 <robot xmlns:xacro="http://www.ros.org/wiki/xacro">
   <xacro:macro name="diffbot" params="prefix">
-  <link name="${prefix}base_link"/>
-  <!-- Was base_link, now body_link -->
-  <link
-    name="${prefix}body_link">
+  <link name="${prefix}base_footprint"/>
+  <link
+    name="${prefix}base_link">
     <inertial>
       <origin
@@ -26,5 +25,5 @@
       <geometry>
         <mesh
-          filename="package://diffdrive_jetbot/description/meshes/body_link.STL" />
+          filename="package://diffdrive_jetbot/description/meshes/base_link.STL" />
       </geometry>
       <material
@@ -40,9 +39,9 @@
       <geometry>
         <mesh
-          filename="package://diffdrive_jetbot/description/meshes/body_link.STL" />
-      </geometry>
-    </collision>
-  </link>
-  <!-- Fixed joint between base_link and body_link -->
+          filename="package://diffdrive_jetbot/description/meshes/base_link.STL" />
+      </geometry>
+    </collision>
+  </link>
+  <!-- Fixed joint between base_footprint and base_link -->
   <joint
     name="${prefix}body_fix_joint"
@@ -52,7 +51,7 @@
       rpy="-1.5708 0 0" />
     <parent
-      link="${prefix}base_link" />
-    <child
-      link="${prefix}body_link" />
+      link="${prefix}base_footprint" />
+    <child
+      link="${prefix}base_link" />
     <axis
       xyz="0 0 0" />
@@ -105,5 +104,5 @@
       rpy="-1.5708 0 3.1416" />
     <parent
-      link="${prefix}body_link" />
+      link="${prefix}base_link" />
     <child
       link="${prefix}caster_ball_link" />
@@ -158,5 +157,5 @@
       rpy="1.9199 -1.5708 3.1416" />
     <parent
-      link="${prefix}body_link" />
+      link="${prefix}base_link" />
     <child
       link="${prefix}camera_link" />
@@ -215,5 +214,5 @@
       rpy="1.5708 0 0" />
     <parent
-      link="${prefix}body_link" />
+      link="${prefix}base_link" />
     <child
       link="${prefix}lidar_link" />
@@ -268,5 +267,5 @@
       rpy="1.5708 0 0" />
     <parent
-      link="${prefix}body_link" />
+      link="${prefix}base_link" />
     <child
       link="${prefix}left_wheel_link" />
@@ -278,20 +277,20 @@
     <inertial>
       <origin
-        xyz="0 0 0"
-        rpy="0 0 0" />
-      <mass
-        value="0" />
-      <inertia
-        ixx="0"
-        ixy="0"
-        ixz="0"
-        iyy="0"
-        iyz="0"
-        izz="0" />
-    </inertial>
-    <visual>
-      <origin
-        xyz="0 0 0"
-        rpy="0 0 0" />
+        xyz="-3.04495944265183E-05 0.0183179040454366 -1.07396547774597E-07"
+        rpy="0 0 0" />
+      <mass
+        value="0.388137366198046" />
+      <inertia
+        ixx="0.000163568162825962"
+        ixy="-1.71522947947033E-07"
+        ixz="-2.55253489205791E-08"
+        iyy="0.000281670214792073"
+        iyz="-1.06397401901507E-09"
+        izz="0.000163656330155147" />
+    </inertial>
+    <visual>
+      <origin
+        xyz="0 0 0"
+        rpy="0 0 3.14359" />
       <geometry>
         <mesh
@@ -307,5 +306,5 @@
       <origin
         xyz="0 0 0"
-        rpy="0 0 0" />
+        rpy="0 0 3.14359" />
       <geometry>
         <mesh
@@ -319,7 +318,7 @@
     <origin
       xyz="0 0 -0.0575"
-      rpy="-1.5708 0 -0.57871" />
-    <parent
-      link="${prefix}body_link" />
+      rpy="-1.5708 3.14359 3.14359" />
+    <parent
+      link="${prefix}base_link" />
     <child
       link="${prefix}right_wheel_link" />

Commit message: fix urdf and adjust correct params for motors

File: src/diffdrive_jetbot/description/ros2_control/diffbot.ros2_control.xacro (robot description, xacro)
@@ -9,5 +9,5 @@
         <param name="device">/dev/ttyMOTOR</param>
         <param name="baud_rate">115200</param>
-        <param name="timeout_ms">20</param>
+        <param name="timeout_ms">10</param>
         <param name="mtype">1</param>
         <param name="deadzone">1600</param>

File: src/diffdrive_jetbot/description/urdf/diffbot.urdf.xacro (robot description, xacro)
@@ -10,5 +10,5 @@
   <!-- Import diffbot ros2_control description -->
   <xacro:include filename="$(find diffdrive_jetbot)/ros2_control/diffbot.ros2_control.xacro" />
-  <xacro:diffbot prefix="$(arg prefix)" />
+  <xacro:diffbot prefix="$(arg prefix)" robot_ip="$(arg robot_ip)" mesh_port="$(arg mesh_port)" />
   <xacro:diffbot_ros2_control
     name="DiffBot" prefix="$(arg prefix)"/>

File: src/diffdrive_jetbot/description/urdf/diffbot_description.urdf.xacro (robot description, xacro)
@@ -1,5 +1,5 @@
 <?xml version="1.0"?>
 <robot xmlns:xacro="http://www.ros.org/wiki/xacro">
-  <xacro:macro name="diffbot" params="prefix">
+  <xacro:macro name="diffbot" params="prefix robot_ip mesh_port">
   <link name="${prefix}base_footprint"/>
   <link
@@ -25,5 +25,5 @@
       <geometry>
         <mesh
-          filename="http://diffbot_ip:8080/meshes/base_link.STL" />
+          filename="http://${robot_ip}:${mesh_port}/meshes/base_link.STL" />
       </geometry>
       <material
@@ -39,5 +39,5 @@
       <geometry>
         <mesh
-          filename="http://diffbot_ip:8080/meshes/base_link.STL" />
+          filename="http://${robot_ip}:${mesh_port}/meshes/base_link.STL" />
       </geometry>
     </collision>
@@ -79,5 +79,5 @@
       <geometry>
         <mesh
-          filename="http://diffbot_ip:8080/meshes/caster_ball_link.STL" />
+          filename="http://${robot_ip}:${mesh_port}/meshes/caster_ball_link.STL" />
       </geometry>
       <material
@@ -93,5 +93,5 @@
       <geometry>
         <mesh
-          filename="http://diffbot_ip:8080/meshes/caster_ball_link.STL" />
+          filename="http://${robot_ip}:${mesh_port}/meshes/caster_ball_link.STL" />
       </geometry>
     </collision>
@@ -132,5 +132,5 @@
       <geometry>
         <mesh
-          filename="http://diffbot_ip:8080/meshes/camera_link.STL" />
+          filename="http://${robot_ip}:${mesh_port}/meshes/camera_link.STL" />
       </geometry>
       <material
@@ -146,5 +146,5 @@
       <geometry>
         <mesh
-          filename="http://diffbot_ip:8080/meshes/camera_link.STL" />
+          filename="http://${robot_ip}:${mesh_port}/meshes/camera_link.STL" />
       </geometry>
     </collision>
@@ -186,5 +186,5 @@
       <geometry>
         <mesh
-          filename="http://diffbot_ip:8080/meshes/lidar_link.STL" />
+          filename="http://${robot_ip}:${mesh_port}/meshes/lidar_link.STL" />
       </geometry>
       <material
@@ -201,5 +201,5 @@
       <geometry>
         <mesh
-          filename="http://diffbot_ip:8080/meshes/lidar_link.STL" />
+          filename="http://${robot_ip}:${mesh_port}/meshes/lidar_link.STL" />
       </geometry>
     </collision>
@@ -242,5 +242,5 @@
       <geometry>
         <mesh
-          filename="http://diffbot_ip:8080/meshes/left_wheel_link.STL" />
+          filename="http://${robot_ip}:${mesh_port}/meshes/left_wheel_link.STL" />
       </geometry>
       <material
@@ -256,5 +256,5 @@
       <geometry>
         <mesh
-          filename="http://diffbot_ip:8080/meshes/left_wheel_link.STL" />
+          filename="http://${robot_ip}:${mesh_port}/meshes/left_wheel_link.STL" />
       </geometry>
     </collision>
@@ -295,5 +295,5 @@
       <geometry>
         <mesh
-          filename="http://diffbot_ip:8080/meshes/right_wheel_link.STL" />
+          filename="http://${robot_ip}:${mesh_port}/meshes/right_wheel_link.STL" />
       </geometry>
       <material
@@ -309,5 +309,5 @@
       <geometry>
         <mesh
-          filename="http://diffbot_ip:8080/meshes/right_wheel_link.STL" />
+          filename="http://${robot_ip}:${mesh_port}/meshes/right_wheel_link.STL" />
       </geometry>
     </collision>
